File: kicad/KoeBlaster/KoeBlaster.kicad_pcb (KiCad board)
At the start: 2 copper layers, 92.5 x 76 mm, 40 parts, among them J1 USB_B_Mini, Q1 BC817, Q2 BC817, Q3 BC817, Q4 BC817, Q5 BC817, SW1 SW_Push, U1 ESP32-WROOM-32, U2 CH340C, U3 NCP1117-3.3_SOT223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

Commit message: various improvements on schematic and pcb
Parts:
- removed Q2, Q4, Q5: BC817, Package_TO_SOT_SMD:SOT-23
- removed SW1: SW_Push, Button_Switch_SMD:SW_SPST_B3U-1000P
- added ?: , , F.Cu at (60.5, 55.0)
- added ?: , , F.Cu at (80.5, 98.0)
- added ?: , , F.Cu at (60.5, 56.5)
- added ?: , , F.Cu at (147.6, 56.5)
- added ?: , , F.Cu at (132.9, 98.5)
- added ?: , , F.Cu at (147.6, 55.0)
- added ?: , , F.Cu at (131.6, 98.5)
- added ?: , , F.Cu at (79.0, 98.0)
- added C8: 1uF, Capacitor_SMD:C_0805_2012Metric_Pad1.18x1.45mm_HandSolder, F.Cu at (104.1, 47.8)
- added C9: 1uF, Capacitor_SMD:C_0805_2012Metric_Pad1.18x1.45mm_HandSolder, F.Cu at (96.6, 88.4)
- added D3: ESD5Z5.0T1G, Diode_SMD:D_SOD-523, F.Cu at (108.4, 98.0)
- added D4: ESD5Z5.0T1G, Diode_SMD:D_SOD-523, F.Cu at (120.7, 97.0)
- added IC1: 74LVC2G14GV,125, SamacSys_Parts:SOT95P275X110-6N, F.Cu at (96.5, 85.1)
- added J2: SJ2-25103A-SMT-TR, SJ2-25103A-SMT-TR:CUI_SJ2-25103A-SMT-TR, B.Cu at (115.0, 99.1)
- added J3: SJ2-25103A-SMT-TR, SJ2-25103A-SMT-TR:CUI_SJ2-25103A-SMT-TR, B.Cu at (126.9, 97.9)
- added Q6: SQ2310CES-T1_GE3, SamacSys_Parts:SOT95P237X112-3N, F.Cu at (85.9, 61.0)
- added R11: 20R, Resistor_SMD:R_0805_2012Metric_Pad1.20x1.40mm_HandSolder, F.Cu at (111.6, 92.0)
- added R15: 10k, Resistor_SMD:R_0805_2012Metric_Pad1.20x1.40mm_HandSolder, F.Cu at (91.4, 59.7)
- added R16: 10k, Resistor_SMD:R_0805_2012Metric_Pad1.20x1.40mm_HandSolder, F.Cu at (100.0, 80.0)
- added R17: 10k, Resistor_SMD:R_0805_2012Metric_Pad1.20x1.40mm_HandSolder, F.Cu at (104.6, 80.0)
- added R9: 20R, Resistor_SMD:R_0805_2012Metric_Pad1.20x1.40mm_HandSolder, F.Cu at (107.6, 92.0)
- added S2: SW_Push, Button_Switch_SMD:SW_SPST_B3U-1000P, F.Cu at (97.8, 51.8)
- C6: value 1uF -> 100nF
- D_FRONT1, D_FRONT2, D_SIDE1, D_SIDE2, D_TOP1: value IR 940nm -> SFH 4547
- Q1: value BC817 -> IRF7324; footprint Package_TO_SOT_SMD:SOT-23 -> Package_SO:SOIC-8_3.9x4.9mm_P1.27mm
- Q3: value BC817 -> BC817DS; footprint Package_TO_SOT_SMD:SOT-23 -> SamacSys_Parts:SOT95P275X110-6N
- R13, R14, R7: value 330R -> 1k
- U4: value TSMP58138 -> TSMP98100
- moved Q3 40.4 mm to (87.6, 76.2)
- moved R14 29.0 mm to (101.6, 86.4), turned to 180 degrees
- moved R13 29.0 mm to (101.6, 83.8), turned to 180 degrees
- moved Q1 24.6 mm to (109.2, 86.4)
- moved R7 18.9 mm to (91.4, 55.9)
- moved R12 13.0 mm to (91.4, 52.1)
- moved C7 11.2 mm to (104.1, 51.4)
- moved R6 8.40 mm to (90.8, 84.2)
- moved R2 7.38 mm to (85.1, 72.4), turned to 180 degrees
- moved C6 6.02 mm to (90.8, 87.0), turned to 180 degrees
- moved R4 5.60 mm to (87.2, 83.2)
- moved R8 3.81 mm to (83.8, 40.6)
- moved U1 2.77 mm to (105.6, 67.7)
- moved C5 1.83 mm to (98.4, 47.8)
- moved R1 0.95 mm to (83.2, 77.5)
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Connections:
- Q1 pad 1: Net-(Q1-B) -> +5V
- Q1 pad 2: Net-(Q1-E) -> Net-(Q1A-G1)
- Q1 pad 3: /EN -> +5V
- Q3 pad 1: Net-(Q3-B) -> Net-(Q3A-E)
- Q3 pad 2: GND -> Net-(Q3A-B)
- Q3 pad 3: Net-(Q3-C) -> /GPIO0
- R1 pad 1: Net-(Q1-B) -> Net-(Q3A-B)
- R1 pad 2: Net-(Q2-E) -> Net-(Q3B-E)
- R10 pad 1: Net-(Q4-C) -> Net-(Q6-D)
- R12 pad 1: Net-(Q5-C) -> Net-(Q6-D)
- R13 pad 1: Net-(Q4-B) -> Net-(Q1A-G1)
- R13 pad 2: /GPIO16 -> Net-(IC1-1Y)
- R14 pad 1: Net-(Q5-B) -> Net-(Q1B-G2)
- R14 pad 2: /GPIO16 -> Net-(IC1-2Y)
- R2 pad 1: Net-(Q2-B) -> Net-(Q3B-B)
- R2 pad 2: Net-(Q1-E) -> Net-(Q3A-E)
- R7 pad 1: Net-(Q3-B) -> Net-(Q6-G)
- R8 pad 1: Net-(Q3-C) -> Net-(Q6-D)
- U1 pad 28: unconnected-(U1-IO17-Pad28) -> /IR_Ext1
- U1 pad 30: unconnected-(U1-IO18-Pad30) -> /IR_Ext2
- U2 pad 13: Net-(Q2-E) -> Net-(Q3B-E)
- U2 pad 14: Net-(Q1-E) -> Net-(Q3A-E)
Routing:
- net Net-(Q6-D): track 0.00 -> 39.5 mm, vias 0 -> 4
- net /GPIO16: track 56.9 -> 28.3 mm, vias 3 -> 2
- net Net-(D4-K): track 0.00 -> 20.6 mm, vias 0 -> 1
- net /IR_Ext2: track 0.00 -> 19.7 mm, vias 0 -> 2
- net Net-(Q5-C): track 17.9 -> 0.00 mm
- net Net-(D_TOP1-K): track 7.18 -> 24.5 mm, vias 0 -> 1
- net Net-(D3-K): track 0.00 -> 14.1 mm, vias 0 -> 1
- net Net-(Q4-B): track 13.4 -> 0.00 mm, vias 2 -> 0
- net Net-(Q1-E): track 12.9 -> 0.00 mm
- net Net-(Q3B-E): track 0.00 -> 11.4 mm
- net Net-(Q3A-E): track 0.00 -> 11.3 mm
- net /IR_Ext1: track 0.00 -> 11.0 mm
- net Net-(Q2-E): track 9.66 -> 0.00 mm
- net Net-(Q1A-D1-Pad7): track 0.00 -> 9.27 mm
- net Net-(Q3-B): track 8.57 -> 0.00 mm
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Other:
- outline, holes or cut-outs redrawn
- board text added: "93°"
- board text added: "98°"

Commit message: prepare everything for hw revision 0.1
Parts:
- added R18: 1k, Resistor_SMD:R_0805_2012Metric_Pad1.20x1.40mm_HandSolder, F.Cu at (98.4, 50.0)
- added R19: 1k, Resistor_SMD:R_0805_2012Metric_Pad1.20x1.40mm_HandSolder, F.Cu at (90.8, 89.8)
- moved S2 5.57 mm to (97.7, 46.2)
- moved C5 4.65 mm to (98.4, 52.5), turned to 0 degrees
- moved R6 1.02 mm to (90.8, 83.2)
- moved R4 1.00 mm to (87.2, 82.2)
- moved C6 0.64 mm to (90.8, 86.4)
Connections:
- net Net-(U2-UD+) renamed /UD+
- net Net-(U2-UD-) renamed /UD-
- S1 pad 2: /GPIO23 -> Net-(S1-N.O.)
- S2 pad 1: /EN -> Net-(R18-Pad1)
Routing:
- net Net-(S1-N.O.): track 0.00 -> 11.3 mm, vias 0 -> 1
- net /GPIO23: track 42.8 -> 31.8 mm, vias 3 -> 2
- net /GPIO27: track 27.9 -> 21.9 mm
- net Net-(R18-Pad1): track 0.00 -> 3.84 mm
- net /UD-: track 37.4 -> 41.1 mm
- net /UD+: track 39.4 -> 42.1 mm
- net /EN: track 53.5 -> 51.6 mm
- net Net-(D_TOP1-K): track 24.5 -> 23.6 mm
- net /GPIO0: track 19.9 -> 19.1 mm
- net GND: vias 32 -> 34

Commit message: updated pcb to v0.2
Parts:
- removed C1: 100nF, Capacitor_SMD:C_0805_2012Metric_Pad1.18x1.45mm_HandSolder
- removed R13, R14, R7: 1k, Resistor_SMD:R_0805_2012Metric_Pad1.20x1.40mm_HandSolder
- Q1: value IRF7324 -> SI9933CDY-T1-GE3
- R10, R8: value 13R -> 5R
- R11, R9: value 20R -> 3R
- R12: value 34R -> 5R
- moved R5 6.78 mm to (92.0, 72.5)
- moved C2 0.47 mm to (69.8, 77.0)
Connections:
- C2 pad 1: Net-(U2-V3) -> +3V3
- J2 pad 3: Net-(D3-K) -> unconnected-(J2-Pad3)
- J3 pad 3: Net-(D4-K) -> unconnected-(J3-Pad3)
- Q1 pad 2: Net-(Q1A-G1) -> Net-(IC1-1Y)
- Q1 pad 4: Net-(Q1B-G2) -> Net-(IC1-2Y)
- Q6 pad 1: Net-(Q6-G) -> /GPIO16
- U2 pad 16: +5V -> +3V3
- U2 pad 4: Net-(U2-V3) -> +3V3
Routing:
- net +3V3: track 109.3 -> 133.8 mm
- net /GPIO2: track 11.9 -> 4.07 mm
- net Net-(IC1-2Y): track 2.96 -> 9.89 mm
- net Net-(IC1-1Y): track 2.96 -> 9.63 mm
- net /GPIO16: track 28.3 -> 34.8 mm
- net Net-(D4-K): track 20.6 -> 14.4 mm
- net Net-(Q6-G): track 6.15 -> 0.00 mm
- net Net-(D3-K): track 14.1 -> 8.05 mm
- net Net-(Q1B-G2): track 4.93 -> 0.00 mm
- net Net-(Q1A-G1): track 4.93 -> 0.00 mm
- net /EN: track 51.6 -> 46.8 mm
- net Net-(U2-V3): track 4.04 -> 0.00 mm
- net +5V: track 200.1 -> 196.5 mm
Other:
- board text added: "KoeBlaster v0.2 04/2024"
- board text removed: "KoeBlaster v0.1 03/2024"
