File: kicad/KoeBlaster/KoeBlaster.kicad_sch (KiCad schematic)
At the start: 40 parts, among them J1 USB_B_Mini, Q1 BC817, Q2 BC817, Q3 BC817, Q4 BC817, Q5 BC817, SW1 SW_Push, U1 ESP32-WROOM-32, U2 CH340C, U3 NCP1117-3.3_SOT223, U4 TSMP58138

Commit message: various improvements on schematic and pcb
Parts:
- removed Q1, Q2, Q3, Q4, Q5: BC817, Package_TO_SOT_SMD:SOT-23, symbol Transistor_BJT:BC817
- added C8, C9: 1uF, Capacitor_SMD:C_0805_2012Metric_Pad1.18x1.45mm_HandSolder, symbol Device:C
- added D3, D4: ESD5Z5.0T1G, Diode_SMD:D_SOD-523, symbol Diode:ESD5Zxx
- added IC1: 74LVC2G14GV,125, SamacSys_Parts:SOT95P275X110-6N, symbol SamacSys_Parts:74LVC2G14GV,125
- added J2, J3: SJ2-25103A-SMT-TR, SJ2-25103A-SMT-TR:CUI_SJ2-25103A-SMT-TR, symbol SJ2-25103A-SMT-TR:SJ2-25103A-SMT-TR
- added Q1: IRF7324, Package_SO:SOIC-8_3.9x4.9mm_P1.27mm, symbol Transistor_FET:IRF7324
- added Q3: BC817DS, SamacSys_Parts:SOT95P275X110-6N, symbol koeblaster_devices:BC817DS_cusom
- added Q6: SQ2310CES-T1_GE3, SamacSys_Parts:SOT95P237X112-3N, symbol SamacSys_Parts:SQ2310CES-T1_GE3
- added R11, R9: 20R, Resistor_SMD:R_0805_2012Metric_Pad1.20x1.40mm_HandSolder, symbol Device:R
- added R15, R16, R17: 10k, Resistor_SMD:R_0805_2012Metric_Pad1.20x1.40mm_HandSolder, symbol Device:R
- C6: value 1uF -> 100nF
- D_FRONT1, D_FRONT2, D_SIDE1, D_SIDE2, D_TOP1: value IR 940nm -> SFH 4547
- J1: footprint 629105150521 -> SamacSys_Parts:629105150521
- R13, R14, R7: value 330R -> 1k
- S2: renamed from SW1; now not fitted
- U4: value TSMP58138 -> TSMP98100; Mouser Part (none) -> https://www.mouser.at/ProductDetail/Vishay-Semiconductors/T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
Connections:
- net +3V3: now also C8.1
- net +5V: now also C9.1, IC1.5 (VCC), Q1.1 (S1), Q1.3 (S2)
- net EN: now also Q3.6 (C)
- net GND: now also C8.2, C9.2, D3.2 (A), D4.2 (A), IC1.2 (GND), J2.1, J2.1.1, J3.1, J3.1.1, Q6.2 (S), R15.2, R16.2, R17.2
- net GPIO0: now also Q3.3 (C)
- net GPIO16: now also R15.1; no longer R13.2, R14.2
- net at R14.1: now also Q1.4 (G2)
- net at R12.1: now also R10.1, R8.1, Q6.3 (D)
- net at R13.1: now also Q1.2 (G1)
- net IR_Ext1: now reaches U1.28 (IO17)
- net IR_Ext1: now also IC1.1 (1A), R16.1
- net IR_Ext2: now reaches U1.30 (IO18)
- net IR_Ext2: now also IC1.3 (2A), R17.1
- net at R2.1: now also Q3.5 (B)
- net at R1.2, U2.13 (~{DTR}): now also Q3.4 (E)
- net at R2.2, U2.14 (~{RTS}): now also Q3.1 (E)
- net at R1.1: now also Q3.2 (B)
- net at R7.1: now also Q6.1 (G)
- new net: D4.1 (K), J3.2, J3.3, R11.1
- new net: D3.1 (K), J2.2, J2.3, R9.1
- new net: Q1.7 (D1), Q1.8 (D1), R9.2
- new net: IC1.4 (2Y), R14.2
- new net: IC1.6 (1Y), R13.2
- new net: Q1.5 (D2), Q1.6 (D2), R11.2
Other:
- note added: "S2 is only used during development to always ensure a proper working reset button. During normal operation S1 should be sufficient. Firmware shall detect short/long press of S1: S1 short: reset blaster S1 long: perform factory reset"
- moved on the sheet: C3, C4, C7, D1, D_FRONT1, D_FRONT2, D_SIDE1, D_SIDE2, D_TOP1, R10, R12, R7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

Commit message: prepare everything for hw revision 0.1
Parts:
- added R18, R19: 1k, Resistor_SMD:R_0805_2012Metric_Pad1.20x1.40mm_HandSolder, symbol Device:R
Connections:
- net EN: now also R18.2; no longer S2.1
- net GPIO23: now also R19.2; no longer S1.2 (N.O.)
- net UD+: now reaches D2.3 (K), J1.3, U2.5 (UD+)
- net UD-: now reaches D2.4 (K), J1.2, U2.6 (UD-)
- new net: R19.1, S1.2 (N.O.)
- new net: R18.1, S2.1
Other:
- note added: "Schematic in evaluation"
- note removed: "Schematic currently under review!"
- moved on the sheet: S1, S2

Commit message: updated pcb to v0.2
Parts:
- removed C1: 100nF, Capacitor_SMD:C_0805_2012Metric_Pad1.18x1.45mm_HandSolder, symbol Device:C
- removed R13, R14, R7: 1k, Resistor_SMD:R_0805_2012Metric_Pad1.20x1.40mm_HandSolder, symbol Device:R
- J2, J3: footprint SJ2-25103A-SMT-TR:CUI_SJ2-25103A-SMT-TR -> CUI_SJ2-25103A-SMT-TR; symbol SJ2-25103A-SMT-TR:SJ2-25103A-SMT-TR -> koeblaster_devices:SJ2-25103A-SMT-TR
- Q1: value IRF7324 -> SI9933CDY-T1-GE3
- R10, R8: value 13R -> 5R
- R11, R9: value 20R -> 3R
- R12: value 34R -> 5R
Connections:
- net +3V3: now also C2.1, U2.16 (VCC), U2.4 (V3)
- net +5V: no longer U2.16 (VCC)
- net GPIO16: now also Q6.1 (G)
- net at D4.1 (K), J3.2, R11.1: no longer J3.3
- net at D3.1 (K), J2.2, R9.1: no longer J2.3
- net at Q1.2 (G1): now also IC1.6 (1Y)
- net at Q1.4 (G2): now also IC1.4 (2Y)
